File: High Resolution Multislope converter-modified rev 2.kicad_pcb (KiCad board)
At the start: 2 copper layers, 100 x 100 mm, 258 parts, among them J1 UART, J2 Input, J3 ICSP6, J4 ISCP10, J5 Power, Q1 BC856, Q2 BC847, Q3 BC856, Q4 BC856, Q5 BC856, Q6 BC856, Q7 BC847, Q8 BC847, Q9 BC856, U1 OPA172, U10 LM393, U11 OPA145, U12 OPA145, U13 MCP6002, U14 7815, U15 7915, U16 LTC2057, U17 74HC74, U18 OPA197, U19 OPA172, U2 OPA172, U20 DG419LDY, U202 MCP4921, U204 ADuM1201AR, U21 OP07CR, U3 7805, U4 NE5534D, U5 74LV4053, U6 LM399H, U7 DG408DJ, U8 OP07CR, U9 OP07CR, X1 16MHz

Commit message: Added silk screen descriptions
All test points and through hole points labeled on front and back

Added test points near to the reference to make it easier to add other references.
Parts:
- removed the REF** at (145.0, 130.5)
- removed the REF** at (145.0, 46.5)
- removed the REF** at (259.5, 123.5)
- removed the REF** at (221.5, 123.5)
- removed the REF** at (174.5, 123.5)
- added +15V: Pin_Header_Straight_1x01_Pitch2.54mm, Pin_Headers:Pin_Header_Straight_1x01_Pitch2.54mm, F.Cu at (76.4, 124.8)
- added +5V: Pin_Header_Straight_1x01_Pitch2.54mm, Pin_Headers:Pin_Header_Straight_1x01_Pitch2.54mm, F.Cu at (20.9, 116.2)
- added -15V: Pin_Header_Straight_1x01_Pitch2.54mm, Pin_Headers:Pin_Header_Straight_1x01_Pitch2.54mm, F.Cu at (78.5, 122.7)
- added GND: Pin_Header_Straight_1x01_Pitch2.54mm, Pin_Headers:Pin_Header_Straight_1x01_Pitch2.54mm, F.Cu at (17.9, 116.2)
- added GNDS: Pin_Header_Straight_1x01_Pitch2.54mm, Pin_Headers:Pin_Header_Straight_1x01_Pitch2.54mm, F.Cu at (70.0, 120.0)
- added GNDS: Pin_Header_Straight_1x01_Pitch2.54mm, Pin_Headers:Pin_Header_Straight_1x01_Pitch2.54mm, F.Cu at (72.1, 122.0)
- added Zener: Pin_Header_Straight_1x01_Pitch2.54mm, Pin_Headers:Pin_Header_Straight_1x01_Pitch2.54mm, F.Cu at (86.9, 107.2)
- moved R8 0.28 mm to (83.2, 110.7)
- moved C20 0.11 mm to (43.2, 132.7)
- moved C44 0.10 mm to (69.0, 132.7)
- moved C23 0.08 mm to (60.4, 132.7)
- moved C204 0.06 mm to (51.8, 132.7)
Routing:
- net GND: track 1284.6 -> 1266.1 mm
- net /U6_15V: track 78.5 -> 87.5 mm
- net -15V: track 443.8 -> 449.0 mm, vias 47 -> 48
- net /U$3_5V: track 21.0 -> 17.2 mm
- net /Integrator_Output: track 74.7 -> 72.8 mm
- net GNDS: track 1511.5 -> 1509.6 mm
- net +15V: track 384.4 -> 386.3 mm
- net Net-(C30-Pad1): track 11.3 -> 10.4 mm
- net /Buffer_Output: track 44.9 -> 44.1 mm
- net +5V: track 448.2 -> 448.9 mm
- net /LM399_Zener_Voltage: track 95.6 -> 96.2 mm
- net /U5_5V: track 16.2 -> 15.6 mm
Other:
- board text added: "+5V"
- board text added: "+Ref"
- board text added: "-Ref"
- board text added: "10 Pin"
- board text added: "16MHz"
- board text added: "5V"
- board text added: "6 Pin"
- board text added: "A+5V"
- board text added: "AC15"
- board text added: "AC5"
- board text added: "ADC0"
- board text added: "ADC1"
- board text added: "AIN0"
- board text added: "AIN1"
- board text added: "AREF"
- board text added: "Buffer Output"
- board text added: "CLK"
- board text added: "Current Mirror Bias Input"
- board text added: "DAC CS"
- board text added: "Enable"
- board text added: "External 10V Reference will need higher voltage"
- board text added: "GND"
- board text added: "IN.1"
- board text added: "IN.2"
- board text added: "IN.3"
- board text added: "IN.4"
- board text added: "IN.6"
- board text added: "Input Switch"
- board text added: "Input Switch Output"
- board text added: "Integrator Input"
- board text added: "Integrator Offset"
- board text added: "Integrator Output"
- board text added: "Jumper for normal use"
- board text added: "MISO"
- board text added: "MOSI"
- board text added: "Microcontroller"
- board text added: "OC1A"
- board text added: "OVER"
- board text added: "PC3"
- board text added: "PC4"
- board text added: "PC5"
- board text added: "PD2"
- board text added: "PD3"
- board text added: "PD4"
- board text added: "PD5"
- board text added: "RST"
- board text added: "RX"
- board text added: "RX_In"
- board text added: "Reference +"
- board text added: "Reference -"
- board text added: "SCLK"
- board text added: "SLV SEL"
- board text added: "SS"
- board text added: "Signal Ground"
- board text added: "Slope Output"
- board text added: "TX"
- board text added: "TX_Out"
- board text added: "Temp Input"
- board text added: "U6_+15V"
- board text added: "Unreg"
- board text added: "VCC"
- board text removed: "EEZ BB3 Plugin Template"

Commit message: Add files via upload
Parts:
- removed +15V, +5V, -15V, GND, Zener: Pin_Header_Straight_1x01_Pitch2.54mm, Pin_Headers:Pin_Header_Straight_1x01_Pitch2.54mm
- removed the GNDS at (70.0, 120.0)
- removed the GNDS at (72.1, 122.0)
- added REF**: SolderWirePad_1x01_Drill2mm, Connector_Wire:SolderWirePad_1x01_Drill2mm, F.Cu at (145.0, 130.5)
- added REF**: SolderWirePad_1x01_Drill2mm, Connector_Wire:SolderWirePad_1x01_Drill2mm, F.Cu at (145.0, 46.5)
- added REF**: PinHeader_2x14_P2.54mm_Horizontal, Connector_PinHeader_2.54mm:PinHeader_2x14_P2.54mm_Horizontal, F.Cu at (259.5, 123.5)
- added REF**: PinHeader_2x14_P2.54mm_Horizontal, Connector_PinHeader_2.54mm:PinHeader_2x14_P2.54mm_Horizontal, F.Cu at (221.5, 123.5)
- added REF**: PinHeader_2x10_P2.54mm_Horizontal, Connector_PinHeader_2.54mm:PinHeader_2x10_P2.54mm_Horizontal, F.Cu at (174.5, 123.5)
- moved R8 0.28 mm to (83.0, 110.5)
- moved C20 0.11 mm to (43.2, 132.8)
- moved C44 0.10 mm to (69.0, 132.8)
- moved C23 0.08 mm to (60.4, 132.8)
- moved C204 0.06 mm to (51.8, 132.8)
Routing:
- net GND: track 1266.1 -> 1284.6 mm
- net /U6_15V: track 87.5 -> 78.5 mm
- net -15V: track 449.0 -> 443.8 mm, vias 48 -> 47
- net /U$3_5V: track 17.2 -> 21.0 mm
- net /Integrator_Output: track 72.8 -> 74.7 mm
- net GNDS: track 1509.6 -> 1511.5 mm
- net +15V: track 386.3 -> 384.4 mm
- net Net-(C30-Pad1): track 10.4 -> 11.3 mm
- net /Buffer_Output: track 44.1 -> 44.9 mm
- net +5V: track 448.9 -> 448.2 mm
- net /LM399_Zener_Voltage: track 96.2 -> 95.6 mm
- net /U5_5V: track 15.6 -> 16.2 mm
Other:
- board text added: "EEZ BB3 Plugin Template"
- board text removed: "+5V"
- board text removed: "+Ref"
- board text removed: "-Ref"
- board text removed: "10 Pin"
- board text removed: "16MHz"
- board text removed: "5V"
- board text removed: "6 Pin"
- board text removed: "A+5V"
- board text removed: "AC15"
- board text removed: "AC5"
- board text removed: "ADC0"
- board text removed: "ADC1"
- board text removed: "AIN0"
- board text removed: "AIN1"
- board text removed: "AREF"
- board text removed: "Buffer Output"
- board text removed: "CLK"
- board text removed: "Current Mirror Bias Input"
- board text removed: "DAC CS"
- board text removed: "Enable"
- board text removed: "External 10V Reference will need higher voltage"
- board text removed: "GND"
- board text removed: "IN.1"
- board text removed: "IN.2"
- board text removed: "IN.3"
- board text removed: "IN.4"
- board text removed: "IN.6"
- board text removed: "Input Switch"
- board text removed: "Input Switch Output"
- board text removed: "Integrator Input"
- board text removed: "Integrator Offset"
- board text removed: "Integrator Output"
- board text removed: "Jumper for normal use"
- board text removed: "MISO"
- board text removed: "MOSI"
- board text removed: "Microcontroller"
- board text removed: "OC1A"
- board text removed: "OVER"
- board text removed: "PC3"
- board text removed: "PC4"
- board text removed: "PC5"
- board text removed: "PD2"
- board text removed: "PD3"
- board text removed: "PD4"
- board text removed: "PD5"
- board text removed: "RST"
- board text removed: "RX"
- board text removed: "RX_In"
- board text removed: "Reference +"
- board text removed: "Reference -"
- board text removed: "SCLK"
- board text removed: "SLV SEL"
- board text removed: "SS"
- board text removed: "Signal Ground"
- board text removed: "Slope Output"
- board text removed: "TX"
- board text removed: "TX_Out"
- board text removed: "Temp Input"
- board text removed: "U6_+15V"
- board text removed: "Unreg"
- board text removed: "VCC"

Commit message: Fix up errors in first fix,
Parts:
- removed the 2-7 at (78.8, 113.1)
- removed the 3-6 at (77.4, 111.7)
- removed the 3-6 at (76.6, 63.0)
- added 3-6: 20K, Resistor_SMD:R_0805_2012Metric, B.Cu at (78.8, 113.0)
- added 3-6: 20K, Resistor_SMD:R_0805_2012Metric, B.Cu at (77.4, 111.7)
- added 3-6: 20K, Resistor_SMD:R_0805_2012Metric, B.Cu at (76.6, 63.0)
Routing:
- net Net-(RN202-Pad7): track 6.78 -> 8.28 mm
- net Net-(RN202-Pad6): track 6.46 -> 7.80 mm
- net /U8_FB: track 15.6 -> 17.0 mm
- net /U9_FB: track 24.0 -> 24.6 mm
- net /Ref_-13.4V: track 120.6 -> 121.3 mm
- net /Ref_+14V: track 182.7 -> 183.4 mm
- net /+Ref_In: track 11.7 -> 12.4 mm
- net /Heater_Setpoint: track 14.9 -> 15.6 mm
- net Net-(R8-Pad1): track 10.9 -> 11.5 mm
